File: ESP32-breakout.kicad_pcb (KiCad board)
At the start: 2 copper layers, 56 parts, among them IC1 ESP32-S2-MINI-2U-N4, J1 UJ20-C-H-G-SMT-1-P16-TR, J2 Conn_01x03, J3 Conn_01x19, J4 Conn_01x19, Q2 Q_NMOS_DGS, SW3 SW_MEC_5E, SW4 SW_MEC_5E, U1 STUSB4500QTR, U2 TJA1051T-3, U4 TPSM33606S3QRDNRQ1, U5 STL6P3LLH6, U6 STL6P3LLH6, U7 MP9361DJ-LF-Z

Commit message: Continued work on the PCB design
Parts:
- C1, C10, C11, C12, C13, C14, C17, C18, C19, C2, C20, C21, C22, C3, C4, C5, C6, C7, C8, C9, CR1, CR2, D1, R1, R11, R12, R14, R15, R16, R17, R2, R3, R4, R5, R6, R7, R8, R9, U2, U7: moved to B.Cu
- moved R1 98.3 mm to (92.7, 125.4)
- moved R15 92.4 mm to (89.2, 125.4)
- moved D1 84.8 mm to (96.5, 130.9)
- moved Q2 83.2 mm to (90.6, 122.5), turned to 90 degrees
- moved C20 83.1 mm to (92.9, 113.7)
- moved C18 82.5 mm to (89.1, 110.9), turned to 180 degrees
- moved CR1 82.3 mm to (93.5, 129.1), turned to 180 degrees
- moved R13 81.0 mm to (97.1, 116.1), turned to 90 degrees
- moved R10 80.7 mm to (93.2, 111.4), turned to 90 degrees
- moved U4 79.6 mm to (89.3, 112.0), turned to -90 degrees
- moved C19 79.2 mm to (89.1, 109.3), turned to 180 degrees
- moved C21 79.0 mm to (89.1, 114.1)
- moved C4 77.5 mm to (94.0, 131.5), turned to -90 degrees
- moved C12 77.4 mm to (99.2, 95.8), turned to 180 degrees
- moved C5 76.2 mm to (96.5, 132.8), turned to 180 degrees
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Connections:
- IC1 pad 10: /LED -> /GPIO 6
- IC1 pad 11: /SCL -> /SDA
- IC1 pad 12: /SDA -> /SCL
- IC1 pad 22: /GPIO 18 -> /LED
- IC1 pad 41: /GPIO 45 -> /CRX_ESP
- IC1 pad 44: /GPIO 46 -> /CTX_ESP
- IC1 pad 8: /CTX_ESP -> /GPIO 4
- IC1 pad 9: /CRX_ESP -> /GPIO 5
- J1 pad A1_B12: (no net) -> GND
- J1 pad A4_B9: (no net) -> VBUS
- J1 pad B1_A12: (no net) -> GND
- J1 pad B4_A9: (no net) -> VBUS
- J3 pad 1: unconnected-(J3-Pin_1-Pad1) -> GND
- J3 pad 10: unconnected-(J3-Pin_10-Pad10) -> /SDA
- J3 pad 11: unconnected-(J3-Pin_11-Pad11) -> /SCL
- J3 pad 12: unconnected-(J3-Pin_12-Pad12) -> /GPIO 9
- J3 pad 13: unconnected-(J3-Pin_13-Pad13) -> /GPIO 10
- J3 pad 14: unconnected-(J3-Pin_14-Pad14) -> /GPIO 11
- J3 pad 15: unconnected-(J3-Pin_15-Pad15) -> /GPIO 12
- J3 pad 16: unconnected-(J3-Pin_16-Pad16) -> /GPIO 13
- J3 pad 17: unconnected-(J3-Pin_17-Pad17) -> /GPIO 14
- J3 pad 18: unconnected-(J3-Pin_18-Pad18) -> /GPIO 15
- J3 pad 19: unconnected-(J3-Pin_19-Pad19) -> /GPIO 16
- J3 pad 2: unconnected-(J3-Pin_2-Pad2) -> +3.3V
- J3 pad 3: unconnected-(J3-Pin_3-Pad3) -> /BOOT
- J3 pad 4: unconnected-(J3-Pin_4-Pad4) -> /GPIO 1
- J3 pad 5: unconnected-(J3-Pin_5-Pad5) -> /GPIO 2
- J3 pad 6: unconnected-(J3-Pin_6-Pad6) -> /GPIO 3
- J3 pad 7: unconnected-(J3-Pin_7-Pad7) -> /GPIO 4
- J3 pad 8: unconnected-(J3-Pin_8-Pad8) -> /GPIO 5
- J3 pad 9: unconnected-(J3-Pin_9-Pad9) -> /GPIO 6
- J4 pad 1: unconnected-(J4-Pin_1-Pad1) -> /CIT_CAN-
- J4 pad 10: unconnected-(J4-Pin_10-Pad10) -> /GPIO 38
- J4 pad 11: unconnected-(J4-Pin_11-Pad11) -> /GPIO 37
- J4 pad 12: unconnected-(J4-Pin_12-Pad12) -> /GPIO 36
- J4 pad 13: unconnected-(J4-Pin_13-Pad13) -> /GPIO 35
- J4 pad 14: unconnected-(J4-Pin_14-Pad14) -> /GPIO 34
- J4 pad 15: unconnected-(J4-Pin_15-Pad15) -> /GPIO 33
- J4 pad 16: unconnected-(J4-Pin_16-Pad16) -> /GPIO 26
- J4 pad 17: unconnected-(J4-Pin_17-Pad17) -> /GPIO 21
- J4 pad 18: unconnected-(J4-Pin_18-Pad18) -> /LED
- J4 pad 19: unconnected-(J4-Pin_19-Pad19) -> /GPIO 17
- J4 pad 2: unconnected-(J4-Pin_2-Pad2) -> /CIT_CAN+
- J4 pad 3: unconnected-(J4-Pin_3-Pad3) -> /EN
- J4 pad 4: unconnected-(J4-Pin_4-Pad4) -> /GPIO 44
- J4 pad 5: unconnected-(J4-Pin_5-Pad5) -> /GPIO 43
- J4 pad 6: unconnected-(J4-Pin_6-Pad6) -> /GPIO 42
- J4 pad 7: unconnected-(J4-Pin_7-Pad7) -> /GPIO 41
- J4 pad 8: unconnected-(J4-Pin_8-Pad8) -> /GPIO 40
- J4 pad 9: unconnected-(J4-Pin_9-Pad9) -> /GPIO 39
- R16 pad 2: /SCL -> /SDA
- R17 pad 2: /SDA -> /SCL
Routing:
- net +3.3V: track 0.00 -> 67.7 mm, vias 0 -> 3
- net /BOOT: track 0.00 -> 40.9 mm, vias 0 -> 3
- net /SDA: track 0.00 -> 37.1 mm, vias 0 -> 2
- net /SCL: track 0.00 -> 37.0 mm, vias 0 -> 2
- net /GPIO 17: track 0.00 -> 33.8 mm, vias 0 -> 1
- net /EN: track 0.00 -> 32.5 mm, vias 0 -> 2
- net VSINK: track 0.00 -> 32.4 mm, vias 0 -> 2
- net /LED: track 0.00 -> 32.0 mm, vias 0 -> 1
- net /GPIO 16: track 0.00 -> 31.2 mm
- net /GPIO 15: track 0.00 -> 26.2 mm, vias 0 -> 1
- net VBUS: track 0.00 -> 26.1 mm, vias 0 -> 3
- net /GPIO 21: track 0.00 -> 24.4 mm, vias 0 -> 1
- net /D+: track 0.00 -> 23.8 mm, vias 0 -> 2
- net /GPIO 13: track 0.00 -> 23.4 mm, vias 0 -> 1
- net /GPIO 14: track 0.00 -> 23.4 mm, vias 0 -> 1
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Other:
- board outline added: 26.4 x 49.3 mm
- copper layers 2 -> 4
