File: _restore_backup_2026-07-19T14-02-08-699/ESP32-breakout.kicad_sch (KiCad schematic)
At the start: 39 parts, among them IC1 ESP32-S2-MINI-2U-N4, J1 UJ20-C-H-G-SMT-1-P16-TR, J2 Conn_01x03, J3 Conn_01x19, J4 Conn_01x19, Q2 Q_NMOS_DGS, SW3 SW_MEC_5E, SW4 SW_MEC_5E, U1 STUSB4500QTR, U2 TJA1051T-3, U4 TPSM33606S3QRDNRQ1, U7 MP9361DJ-LF-Z

Commit message: Continued work on the PCB design
Connections:
- net +3.3V: no longer J3.2 (Pin_2)
- net BOOT: no longer J3.3 (Pin_3)
- net CIT_CAN+: no longer J4.2 (Pin_2)
- net CIT_CAN-: no longer J4.1 (Pin_1)
- net CRX_ESP: now also IC1.9 (IO5); no longer IC1.41 (IO45)
- net CTX_ESP: now also IC1.8 (IO4); no longer IC1.44 (IO46)
- net EN: no longer J4.3 (Pin_3)
- net GND: now also J1.A1 (GND), J1.A12 (GND), J1.B1 (GND), J1.B12 (GND), J1.S1 (SHIELD); no longer J1.A1_B12 (GND), J1.B1_A12 (GND), J1.SH (SHIELD), J3.1 (Pin_1)
- net GPIO 1: no longer J3.4 (Pin_4)
- net GPIO 10: no longer J3.13 (Pin_13)
- net GPIO 11: no longer J3.14 (Pin_14)
- net GPIO 12: no longer J3.15 (Pin_15)
- net GPIO 13: no longer J3.16 (Pin_16)
- net GPIO 14: no longer J3.17 (Pin_17)
- net GPIO 15: no longer J3.18 (Pin_18)
- net GPIO 16: no longer J3.19 (Pin_19)
- net GPIO 17: no longer J4.19 (Pin_19)
- net GPIO 2: no longer J3.5 (Pin_5)
- net GPIO 21: no longer J4.17 (Pin_17)
- net GPIO 26: no longer J4.16 (Pin_16)
- net GPIO 3: no longer J3.6 (Pin_6)
- net GPIO 33: no longer J4.15 (Pin_15)
- net GPIO 34: no longer J4.14 (Pin_14)
- net GPIO 35: no longer J4.13 (Pin_13)
- net GPIO 36: no longer J4.12 (Pin_12)
- net GPIO 37: no longer J4.11 (Pin_11)
- net GPIO 38: no longer J4.10 (Pin_10)
- net GPIO 39: no longer J4.9 (Pin_9)
- net GPIO 40: no longer J4.8 (Pin_8)
- net GPIO 41: no longer J4.7 (Pin_7)
- net GPIO 42: no longer J4.6 (Pin_6)
- net GPIO 43: no longer J4.5 (Pin_5)
- net GPIO 44: no longer J4.4 (Pin_4)
- net GPIO 9: no longer J3.12 (Pin_12)
- net LED: now also IC1.10 (IO6); no longer IC1.22 (IO18), J4.18 (Pin_18)
- net SCL: now also IC1.11 (IO7), R16.2; no longer IC1.12 (IO8), J3.11 (Pin_11), R17.2
- net SDA: now also IC1.12 (IO8), R17.2; no longer IC1.11 (IO7), J3.10 (Pin_10), R16.2
- net VBUS: now also J1.A4 (VBUS), J1.A9 (VBUS), J1.B4 (VBUS), J1.B9 (VBUS); no longer J1.A4_B9 (VBUS), J1.B4_A9 (VBUS)
- net GPIO 4: no longer names the net of J3.7 (Pin_7)
- net GPIO 4: no longer IC1.8 (IO4)
- net GPIO 5: no longer names the net of J3.8 (Pin_8)
- net GPIO 5: no longer IC1.9 (IO5)
- net GPIO 6: no longer names the net of J3.9 (Pin_9)
- net GPIO 6: no longer IC1.10 (IO6)
- new net GPIO 18: IC1.22 (IO18)
- new net GPIO 45: IC1.41 (IO45)
- new net GPIO 46: IC1.44 (IO46)
Other:
- moved on the sheet: J1, J4
