File: _restore_backup_2026-08-08T16-09-21-337/ESP32-breakout.kicad_pcb (KiCad board)
At the start: 4 copper layers, 26.4 x 49.3 mm, 56 parts, among them IC1 ESP32-S2-MINI-2U-N4, J1 UJ20-C-H-G-SMT-1-P16-TR, J2 Conn_01x03, J3 Conn_01x19, J4 Conn_01x19, Q2 Q_NMOS_DGS, SW3 SW_MEC_5E, SW4 SW_MEC_5E, U1 STUSB4500QTR, U2 TJA1051T-3, U4 TPSM33606S3QRDNRQ1, U5 STL6P3LLH6, U6 STL6P3LLH6, U7 MP9361DJ-LF-Z

Commit message: Finished first revision of PCB
Parts:
- moved CR1 0.36 mm to (93.5, 129.1)
Routing:
- net GND: vias 8 -> 7
